Commit message: I have added the basic structure of the bot

File: src/my_robot_description/urdf/my_robot.urdf (robot description, URDF)
Before this commit: robot my_robot, 1 links, 0 joints
Links:
- added link caster_wheel_link; visual sphere radius=0.075
- added link left_wheel_link; visual cylinder length=0.05 radius=0.15
- added link right_wheel_link; visual cylinder length=0.05 radius=0.15
- link base_link: geometry visual box size=0.6 0.4 0.2
Joints:
- added joint base_caster_wheel_joint: type fixed, parent base_link, child caster_wheel_link, origin xyz=0.225 0 -0.075 rpy=0 0 0
- added joint base_left_wheel_joint: type continuous, parent base_link, child left_wheel_link, origin xyz=-0.15 0.2 0 rpy=1.57 0 0, axis 0 0 1
- added joint base_right_wheel_joint: type continuous, parent base_link, child right_wheel_link, origin xyz=-0.15 -0.2 0 rpy=1.57 0 0, axis  0 0 1

Commit message: The basic structure of the BOT

File: src/my_robot_description/urdf/my_robot.urdf (robot description, URDF)
Before this commit: robot my_robot, 4 links, 3 joints
Links:
- added link base_footprint
Joints:
- added joint base_footprint_joint: type fixed, parent base_footprint, child base_link, origin xyz=0 0 0.15 rpy=0 0 0
- joint base_left_wheel_joint: axis 0 0 1 -> 0 1 0; origin xyz=-0.15 0.2 0 rpy=1.57 0 0 -> xyz=-0.15 0.2 0 rpy=0 0 0
- joint base_right_wheel_joint: axis  0 0 1 ->  0 1 0; origin xyz=-0.15 -0.2 0 rpy=1.57 0 0 -> xyz=-0.15 -0.2 0 rpy=0 0 0
