Commit message: Added Inertial and collision tag

File: src/my_robot_description/urdf/common_properties.xacro (robot description, xacro)
@@ -16,3 +16,49 @@
     <xacro:property name="wheel_length" value="0.05"/>
     <xacro:property name="caster_wheel_radius" value="${wheel_radius/2}"/>
+    <xacro:macro name="box_inertia" params="m l b h xyz rpy">
+        <inertial>
+            <origin xyz="${xyz}" rpy="${rpy}"/>
+            <mass value="${m}"/>
+            <inertia ixx="${(1/12)*m*(h*h + l*l)}" ixy="0" ixz="0"
+                     iyy="${(1/12)*m*(b*b + l*l)}" iyz="0"
+                     izz="${(1/12)*m*(b*b + h*h)}"/>
+        </inertial>
+    </xacro:macro>
+    <xacro:macro name="wheel_inertia" params="m l r xyz rpy">
+        <inertial>
+            <origin xyz="${xyz}" rpy="${rpy}"/>
+            <mass value="${m}"/>
+            <inertia ixx="${(1/12)*m*((3*r*r) + l*l)}" ixy="0" ixz="0"
+                     iyy="${(1/12)*m*((3*r*r) + l*l)}" iyz="0"
+                     izz="${(1/2)*m*r*r}"/>
+        </inertial>
+    </xacro:macro>
+    <xacro:macro name="sphere_inertia" params="m r xyz rpy">
+        <inertial>
+            <origin xyz="${xyz}" rpy="${rpy}"/>
+            <mass value="${m}"/>
+            <inertia ixx="${(2/5)*m*r*r}" ixy="0" ixz="0"
+                     iyy="${(2/5)*m*r*r}" iyz="0"
+                     izz="${(2/5)*m*r*r}"/>
+        </inertial>
+    </xacro:macro>
+    <xacro:macro name="wheel_link" params="prefix y">
+        <link name="${prefix}_wheel_link">
+            <visual>
+                <geometry>
+                    <cylinder radius="${wheel_radius}" length="${wheel_length}"/>
+                </geometry>
+                <origin xyz="0 ${y} 0" rpy="${pi/2} 0 0"/>
+                <material name="blue"/>
+            </visual>
+            <collision>
+                <geometry>
+                    <cylinder radius="${wheel_radius}" length="${wheel_length}"/>
+                </geometry>
+                <origin xyz="0 ${y} 0" rpy="${pi/2} 0 0"/>
+            </collision>
+            <xacro:wheel_inertia m="1.0" l="${wheel_length}" r="${wheel_radius}"
+                                 xyz="0 ${y} 0" rpy="${pi/2} 0 0"/>
+        </link>
+    </xacro:macro>
 </robot>

File: src/my_robot_description/urdf/mobile_base.xacro (robot description, xacro)
@@ -10,16 +10,13 @@
             <material name="red"/>
         </visual>
+        <collision>
+            <geometry>
+                <box size="${base_length} ${base_breadth} ${base_height}"/>
+            </geometry>
+            <origin xyz="0 0 ${base_height/2}" rpy="0 0 0"/>
+        </collision>
+        <xacro:box_inertia m="5.0" l="${base_length}" b="${base_breadth}" h="${base_height}"
+                           xyz="0 0 ${base_height/2}" rpy="0 0 0"/>
     </link>
-    <xacro:macro name="wheel_link" params="prefix y">
-        <link name="${prefix}_wheel_link">
-            <visual>
-                <geometry>
-                    <cylinder radius="${wheel_radius}" length="${wheel_length}"/>
-                </geometry>
-                <origin xyz="0 ${y} 0" rpy="${pi/2} 0 0"/>
-                <material name="blue"/>
-            </visual>
-        </link>
-    </xacro:macro>
     <xacro:wheel_link prefix="right" y="-${wheel_length/2}"/>
     <xacro:wheel_link prefix="left" y="${wheel_length/2}"/>
@@ -29,6 +26,15 @@
                 <sphere radius="${caster_wheel_radius}"/>
             </geometry>
+            <origin xyz="0 0 0" rpy="0 0 0"/>
             <material name="green"/>
         </visual>
+        <collision>
+            <geometry>
+                <sphere radius="${caster_wheel_radius}"/>
+            </geometry>
+            <origin xyz="0 0 0" rpy="0 0 0"/>
+        </collision>
+        <xacro:sphere_inertia m="0.5" r="${caster_wheel_radius}"
+                              xyz="0 0 0" rpy="0 0 0"/>
     </link>
     <joint name="base_footprint_joint" type="fixed">

Commit message: Add few stuffs

File: src/my_robot_description/urdf/common_properties.xacro (robot description, xacro)
@@ -9,4 +9,7 @@
     <material name="blue">
         <color rgba="0 0 1 1"/>
+    </material>
+    <material name="grey">
+        <color rgba="0.5 0.5 0.5 1"/>
     </material>
     <xacro:property name="base_length" value="0.6"/>
@@ -58,5 +61,5 @@
                 <origin xyz="0 ${y} 0" rpy="${pi/2} 0 0"/>
             </collision>
-            <xacro:wheel_inertia m="1.0" l="${wheel_length}" r="${wheel_radius}"
+            <xacro:wheel_inertia m="1.0" l="${2*wheel_length}" r="${2*wheel_radius}"
                                  xyz="0 ${y} 0" rpy="${pi/2} 0 0"/>
         </link>

File: src/my_robot_description/urdf/mobile_base.xacro (robot description, xacro)
@@ -16,5 +16,5 @@
             <origin xyz="0 0 ${base_height/2}" rpy="0 0 0"/>
         </collision>
-        <xacro:box_inertia m="5.0" l="${base_length}" b="${base_breadth}" h="${base_height}"
+        <xacro:box_inertia m="5.0" l="${2*base_length}" b="${2*base_breadth}" h="${2*base_height}"
                            xyz="0 0 ${base_height/2}" rpy="0 0 0"/>
     </link>
@@ -35,5 +35,5 @@
             <origin xyz="0 0 0" rpy="0 0 0"/>
         </collision>
-        <xacro:sphere_inertia m="0.5" r="${caster_wheel_radius}"
+        <xacro:sphere_inertia m="0.5" r="${2*caster_wheel_radius}"
                               xyz="0 0 0" rpy="0 0 0"/>
     </link>

File: src/my_robot_description/urdf/my_robot.urdf.xacro (robot description, xacro)
@@ -3,3 +3,5 @@
     <xacro:include filename="common_properties.xacro"/>
     <xacro:include filename="mobile_base.xacro"/>
+    <xacro:include filename="mobile_base_gazebo.xacro"/>
+    <xacro:include filename="camera.xacro"/>
 </robot>
